File: Kicad/Tocadiscos_RFID/Tocadiscos_RFID.kicad_sch (KiCad schematic)
At the start: 6 parts, among them M1 Stepper_Motor_unipolar_5pin, P1 Conn_02x20, P2 Conn_02x20, U1 DFPlayer_MiniMP3, U2 ULN2003

Commit message: Algunos pines
Parts:
- added D1: OLED Display, Display:OLED-128O064D, symbol MCE_Displays:OLED_Display128x64
Changed lines of the file:
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@@
+	)
+	(symbol
+		(lib_id "MCE_Displays:OLED_Display128x64")
+		(at 93.98 121.92 0)
+		(unit 1)
+		(body_style 1)
+		(exclude_from_sim no)
+		(in_bom yes)
+		(on_board yes)
+		(in_pos_files yes)
+		(dnp no)
+		(fields_autoplaced yes)
+		(property "Reference" "D1"
+			(at 102.87 120.6499 0)
+			(show_name no)
+			(do_not_autoplace no)
+			(effects
+				(font
+					(size 1.27 1.27)
+				)
+				(justify left)
+			)
+		)
+		(property "Value" "OLED Display"
+			(at 102.87 123.1899 0)
+			(show_name no)
+			(do_not_autoplace no)
+			(effects
+				(font
+					(size 1.27 1.27)
+				)
+				(justify left)
+			)
+		)
+		(property "Footprint" "Display:OLED-128O064D"
+			(at 93.98 121.92 0)
+			(hide yes)
+			(show_name no)
+			(do_not_autoplace no)
+			(effects
+				(font
+					(size 1.27 1.27)
+				)
+			)
+		)
+		(property "Datasheet" ""
+			(at 93.98 121.92 0)
+			(hide yes)
+			(show_name no)
+			(do_not_autoplace no)
+			(effects
+				(font
+					(size 1.27 1.27)
+				)
+			)
+		)
+		(property "Description" "Modulo de pantalla OLED"
+			(at 94.488 137.922 0)
+			(hide yes)
+			(show_name no)
+			(do_not_autoplace no)
+			(effects
+				(font
+					(size 1.27 1.27)
+				)
+			)
+		)
+		(pin "2"
+		)
+		(pin "4"
+		)
+		(pin "1"
+		)
+		(pin "3"
+		)
+		(instances
+			(project "Tocadiscos_RFID"
+				(path "/75ce41c1-38be-4585-ae72-3abeaf0221a7"
+					(reference "D1")
+					(unit 1)
+				)
+			)
+		)
 	)
 	(symbol

Commit message: pines del motor(que seguro hay que cambiar)
Connections:
- net SPI_MISO: now reaches P2.18 (Pin_18)
- net SPI_MISO: now also RFID1.4 (MISO)
- net SPI_SCK: now reaches P2.20 (Pin_20)
- net SPI_SCK: now also RFID1.2 (SCK)
- net SPI_MOSI: now reaches P2.21 (Pin_21)
- net SPI_MOSI: now also RFID1.3 (MOSI)
- net RFID_RST: now reaches P2.29 (Pin_29)
- net RFID_RST: now also RFID1.7 (RST)
- net RFID_CS: now reaches P2.31 (Pin_31)
- net RFID_CS: now also RFID1.1 (SDA)
- net MOTOR_IN1: now reaches P2.32 (Pin_32)
- net MOTOR_IN1: now also U2.1 (I1)
- net MOTOR_IN2: now reaches P2.34 (Pin_34)
- net MOTOR_IN2: now also U2.2 (I2)
- net MOTOR_IN3: now reaches P2.36 (Pin_36)
- net MOTOR_IN3: now also U2.3 (I3)
- net MOTOR_IN4: now reaches P2.38 (Pin_38)
- net MOTOR_IN4: now also U2.4 (I4)
- net I2C_SCL: now reaches D1.3 (SCL)
- net I2C_SCL: now also P1.21 (Pin_21)
- net I2C_SDA: now reaches D1.4 (SDA)
- net I2C_SDA: now also P1.19 (Pin_19)
- net UART_RX: now reaches P1.23 (Pin_23)
- net UART_RX: now also U1.3 (TX)
- net UART_TX: now reaches P1.25 (Pin_25)
- net UART_TX: now also U1.2 (RX)
Other:
- moved on the sheet: D1, M1, RFID1, U1, U2

Commit message: nada
Parts:
- D1: value OLED Display -> OLED 1.3" SH1106
Connections:
- net +3V3: now reaches P2.1 (Pin_1)
- net +3V3: now also D1.2 (VCC), RFID1.8 (VCC)
- net +5V: now reaches P2.2 (Pin_2)
- net +5V: now also U1.1 (VCC)
- net GND: now reaches P2.39 (Pin_39)
- net GND: now also D1.1 (GND), RFID1.6 (GND), U1.10 (GND), U1.7 (GND)
- no-connect marks 0 -> 1
Other:
- moved on the sheet: D1, U1

Commit message: .
Parts:
- added LS1: Speaker 4R 3W, Package_SON:WSON-8-1EP_6x5mm_P1.27mm_EP3.4x4mm, symbol Device:Speaker
Connections:
- net at U1.6 (SPK1(+)): now also LS1.1
- net at U1.8 (SPK2(-)): now also LS1.2
- no-connect marks 1 -> 7
Other:
- note added: "Se puede usar como señal de control"
- note added: "Tienen resistencias pull-up internas"
- moved on the sheet: M1, P1, U2
